File: PCBs/din8_de9/PC8801UNIV_DIN8_DE9.kicad_pcb (KiCad board)
At the start: 2 copper layers, 219 x 95 mm, 1783 parts, among them J1 PC8801EXT, J2 Conn_02x36_Odd_Even, J3 Conn_02x36_Odd_Even, J4 DIN8, J5 DSUB-9_Male_Horizontal_P2.77x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

Commit message: ライセンス明記、
Parts:
- added REF**: OSHW-Logo2_7.3x6mm_SilkScreen, Symbol:OSHW-Logo2_7.3x6mm_SilkScreen, F.Cu at (50.3, 119.9)
Other:
- board text added: "Licensed under CERN-OHL-W v2"
